Commit message: Fix camera link position Add camera link color

File: urdf/dumpster.xacro (robot description, xacro)
@@ -224,12 +224,12 @@
       <origin xyz="0.0 0 0" rpy="0 0 0"/>
       <geometry>
-         <box size="0.05 0.05 0.05"/>
+         <box size="0.025 0.05 0.05"/>
       </geometry>
     </visual>
   </link>
 <joint type="fixed" name="camera_joint">
-    <origin xyz="0.2 0 0" rpy="0 0 0"/>
+    <origin xyz="0.0375 0 0.224" rpy="0 0 0"/>
     <child link="camera"/>
-    <parent link="chassis"/>
+    <parent link="laser_pole"/>
   </joint>
 <!-- Laser -->

Commit message: Add launch node for Rviz with basic config file Add basic Rviz configuration file Fix Rviz crash due to model with stl mesh file: - Add dump bin mesh file in dae (collada) format - Edit robot xacro file to use collada file format Comment robot_description launch file

File: urdf/dumpster.xacro (robot description, xacro)
@@ -60,5 +60,4 @@
   </link>
 <!-- Dump box -->
-<!--  -->
     <joint name="dump_box_joint" type="fixed">
     <origin xyz="0 0 0.1" rpy="1.57079 0 1.57079" />
@@ -86,9 +85,9 @@
       <origin xyz="-0.355 -0.05 0.2" rpy=" 0 0 0"/>
         <geometry>
-        <mesh filename="package://dumpster/meshes/dumper_bin.stl" scale="0.006 0.006 0.006"/>
+        <mesh filename="package://dumpster/meshes/dumper_bin.dae" scale="0.006 0.006 0.006"/>
         </geometry>
         <material name="blue"/>
     </visual>
-  </link>
+ </link>
 <!-- plastic bin -->
 <!--

Commit message: Fix issue 'robot does not move when cmd_vel is published': - Edit robot model collision geometry, mass value and position of links

File: urdf/dumpster.xacro (robot description, xacro)
@@ -2,8 +2,6 @@
 <robot name="dumpster" xmlns:xacro="http://www.ros.org/wiki/xacro">
 <xacro:include filename="$(find dumpster)/urdf/dumpster.gazebo" />
-<material name="blue">
-      <color rgba="0 0 0.8 1"/>
-</material>
   <link name="robot_footprint"></link>
+<!-- Chassis & caster wheels -->
   <joint name="robot_footprint_joint" type="fixed">
     <origin xyz="0 0 0" rpy="0 0 0" />
@@ -12,8 +10,8 @@
   </joint>
   <link name='chassis'>
-    <pose>0 0 0 0 0 0</pose>
+    <pose>0 0 0.15 0 0 0</pose>
     <inertial>
       <mass value="15.0"/>
-      <origin xyz="0.1 0 0" rpy=" 0 0 0"/>
+      <origin xyz="0.0 0 0" rpy=" 0 0 0"/>
       <inertia
           ixx="0.1" ixy="0" ixz="0"
@@ -23,5 +21,5 @@
     </inertial>
     <collision name='collision'>
-      <origin xyz="0.1 0 0" rpy=" 0 0 0"/>
+      <origin xyz="0.0 0 0" rpy=" 0 0 0"/>
       <geometry>
         <box size=".6 .4 .1"/>
@@ -29,5 +27,5 @@
     </collision>
     <visual name='chassis_visual'>
-      <origin xyz="0.1 0 0" rpy=" 0 0 0"/>
+      <origin xyz="0.0 0 0" rpy=" 0 0 0"/>
       <geometry>
         <box size=".6 .4 .1"/>
@@ -35,5 +33,5 @@
     </visual>
     <collision name='back_caster_collision'>
-      <origin xyz="-0.15 0 -0.1" rpy=" 0 0 0"/>
+      <origin xyz="-0.25 0 -0.1" rpy=" 0 0 0"/>
       <geometry>
         <sphere radius="0.0499"/>
@@ -41,5 +39,5 @@
     </collision>
     <visual name='back_caster_visual'>
-      <origin xyz="-0.15 0 -0.1" rpy=" 0 0 0"/>
+      <origin xyz="-0.25 0 -0.1" rpy=" 0 0 0"/>
       <geometry>
         <sphere radius="0.05"/>
@@ -47,5 +45,5 @@
     </visual>
     <collision name='front_caster_collision'>
-      <origin xyz="0.3 0 -0.1" rpy=" 0 0 0"/>
+      <origin xyz="0.25 0 -0.1" rpy=" 0 0 0"/>
       <geometry>
         <sphere radius="0.0499"/>
@@ -53,5 +51,5 @@
     </collision>
     <visual name='front_caster_visual'>
-      <origin xyz="0.3 0 -0.1" rpy=" 0 0 0"/>
+      <origin xyz="0.25 0 -0.1" rpy=" 0 0 0"/>
       <geometry>
         <sphere radius="0.05"/>
@@ -68,6 +66,6 @@
     <pose>0 0 0 0 0 0</pose>
     <inertial>
-      <mass value="15.0"/>
-      <origin xyz="0.0 0 0" rpy=" 0 0 0"/>
+      <mass value="0.0"/>
+      <origin xyz="0 0 -0.1" rpy=" 0 0 0"/>
       <inertia
           ixx="0.1" ixy="0" ixz="0"
@@ -77,19 +75,18 @@
     </inertial>
     <collision name='collision'>
-      <origin xyz="0 0.0 0.1" rpy=" 0 0 0"/>
-      <geometry>
-        <box size=".8 .4 .1"/>
+      <origin xyz="0 0 -0.1" rpy=" 0 0 0"/>
+      <geometry>
+        <box size=".1 .1 .1"/>
       </geometry>
     </collision>
     <visual name='dump_box_visual'>
-      <origin xyz="-0.355 -0.05 0.2" rpy=" 0 0 0"/>
+      <origin xyz="-0.355 -0.05 0.1" rpy=" 0 0 0"/>
         <geometry>
         <mesh filename="package://dumpster/meshes/dumper_bin.dae" scale="0.006 0.006 0.006"/>
         </geometry>
-        <material name="blue"/>
     </visual>
  </link>
 <!-- plastic bin -->
-<!--
+  <!--
     <joint name="plastic_bin_joint" type="fixed">
  <origin xyz="0.0 0.0 0.0" rpy="0 0 -1.57079" />
@@ -109,5 +106,5 @@
 <!-- laser pole -->
 <joint type="fixed" name="pole_joint">
-    <origin xyz="0.35 0.0 0.1" rpy="0 0 0"/>
+    <origin xyz="0.25 0.0 0.1" rpy="0 0 0"/>
     <child link="laser_pole"/>
     <parent link="chassis"/>
@@ -116,5 +113,5 @@
     <pose>0 0 0 0 0 0</pose>
     <inertial>
-      <mass value="15.0"/>
+      <mass value="0.2"/>
       <origin xyz="0.0 0 0" rpy=" 0 0 0"/>
       <inertia
@@ -127,5 +124,5 @@
       <origin xyz="0 0.0 0.1" rpy=" 0 0 0"/>
       <geometry>
-        <box size=".8 .4 .1"/>
+        <box size="0.05 0.05 0.3"/>
       </geometry>
     </collision>
@@ -147,5 +144,5 @@
   </joint>
 <link name='left_wheel'>
-    <pose>0 0 0.1 0 0 0</pose>
+    <pose>0 0 0.15 0 0 0</pose>
     <inertial>
       <mass value="5.0"/>
@@ -179,5 +176,5 @@
   </joint>
 <link name='right_wheel'>
-    <pose>0 0 0.1 0 0 0</pose>
+    <pose>0 0 0.15 0 0 0</pose>
     <inertial>
       <mass value="5.0"/>
@@ -234,5 +231,5 @@
 <!-- Laser -->
 <link name="hokuyo">
-    <pose>0 0 0.5 0 0 0</pose>
+    <pose>0 0 0.1 0 0 0</pose>
     <inertial>
       <mass value="0.1"/>
@@ -251,12 +248,12 @@
     </collision>
     <visual name='hokuyo_visual'>
-      <origin xyz="0.0 0 -0.05" rpy="0 0 0"/>
-      <geometry>
-         <mesh filename="package://dumpster/meshes/hokuyo.dae"/>
+      <origin xyz="0.0 0 0" rpy="0 0 0"/>
+      <geometry>
+         <mesh filename="package://udacity_bot/meshes/hokuyo.dae"/>
       </geometry>
     </visual>
   </link>
 <joint type="fixed" name="hokuyo_joint">
-    <origin xyz="0.0 0 0.335" rpy="0 0 0"/>
+    <origin xyz="0.0 0 0.285" rpy="0 0 0"/>
     <child link="hokuyo"/>
     <parent link="laser_pole"/>
