Commit message: Rename package name from dumpster to rtab_dumpster Rename in all file names and file content all instances of 'dumpster' to 'rtab_dumpster'

File: urdf/rtab_dumpster.xacro (robot description, xacro)
@@ -1,5 +1,5 @@
 <?xml version='1.0'?>
-<robot name="dumpster" xmlns:xacro="http://www.ros.org/wiki/xacro">
-<xacro:include filename="$(find dumpster)/urdf/dumpster.gazebo" />
+<robot name="rtab_dumpster" xmlns:xacro="http://www.ros.org/wiki/xacro">
+<xacro:include filename="$(find rtab_dumpster)/urdf/rtab_dumpster.gazebo" />
   <link name="robot_footprint"></link>
 <!-- Chassis & caster wheels -->
@@ -83,5 +83,5 @@
       <origin xyz="-0.355 -0.05 0.1" rpy=" 0 0 0"/>
         <geometry>
-        <mesh filename="package://dumpster/meshes/dumper_bin.dae" scale="0.006 0.006 0.006"/>
+        <mesh filename="package://rtab_dumpster/meshes/dumper_bin.dae" scale="0.006 0.006 0.006"/>
         </geometry>
     </visual>
@@ -99,5 +99,5 @@
      <origin xyz="-0.319 -1.895 -0.285" rpy=" 0 0 0"/>
           <geometry>
-            <mesh filename="package://dumpster/meshes/plastic_bin_bin.stl" scale="0.14 0.14 0.14"/>
+            <mesh filename="package://rtab_dumpster/meshes/plastic_bin_bin.stl" scale="0.14 0.14 0.14"/>
           </geometry>
         </visual>
@@ -250,5 +250,5 @@
       <origin xyz="0.0 0 0" rpy="0 0 0"/>
       <geometry>
-         <mesh filename="package://udacity_bot/meshes/hokuyo.dae"/>
+         <mesh filename="package://rtab_dumpster/meshes/hokuyo.dae"/>
       </geometry>
     </visual>

Commit message: Add Gazebo plugin for depth camera

File: urdf/rtab_dumpster.xacro (robot description, xacro)
@@ -200,5 +200,5 @@
   </link>
 <!-- Camera -->
-<link name="camera">
+<link name="camera"> <!-- must match the name of the reference in the .gazebo file -->
     <pose>0 0 0.1 0 0 0</pose>
     <inertial>

Commit message: Add Kinect Sensor to robot urdf model Add meshes and textures of Kinect Sensor Comment out hokuyo laser and camera from robot urdf model

File: urdf/rtab_dumpster.xacro (robot description, xacro)
@@ -200,5 +200,7 @@
   </link>
 <!-- Camera -->
-<link name="camera"> <!-- must match the name of the reference in the .gazebo file -->
+<!-- link name must match the name of the reference in the .gazebo file -->
+<!--
+<link name="camera">
     <pose>0 0 0.1 0 0 0</pose>
     <inertial>
@@ -229,5 +231,22 @@
     <parent link="laser_pole"/>
   </joint>
+-->
+<!-- Kinect Sensor -->
+<!-- link name must match the name of the reference in the .gazebo file -->
+    <link name="kinect_link">
+        <visual>
+            <origin xyz="0 0 0" rpy="0 0 1.5708"/>
+            <geometry>
+                <mesh filename="package://rtab_dumpster/meshes/kinect.dae" scale="1.0 1.0 1.0"/>
+            </geometry>
+        </visual>
+    </link>
+    <joint name="kinect_joint" type="fixed">
+        <origin xyz="0.0 0 0.285" rpy="0 0 0"/>
+        <parent link="laser_pole"/>
+        <child link="kinect_link"/>
+</joint>
 <!-- Laser -->
+<!--
 <link name="hokuyo">
     <pose>0 0 0.1 0 0 0</pose>
@@ -259,3 +278,4 @@
     <parent link="laser_pole"/>
   </joint>
+-->
 </robot>

Commit message: Add Kinect Sensor as external xacro file (include) Add camera_rgb_joint, camera_rgb_frame (link) Add camera_rgb_optical_joint, camera_rgb_optical_frame (link) Add camera_depth_joint, camera_depth_frame (link) Add camera_joint, camera_link (frame) Delete Kinect Sensor code from rtab_dumpster.xacro

File: urdf/rtab_dumpster.xacro (robot description, xacro)
@@ -104,11 +104,11 @@
       </link>
 -->
-<!-- laser pole -->
-<joint type="fixed" name="pole_joint">
-    <origin xyz="0.25 0.0 0.1" rpy="0 0 0"/>
-    <child link="laser_pole"/>
-    <parent link="chassis"/>
-  </joint>
-  <link name='laser_pole'>
+<!-- kinect pole -->
+<joint type="fixed" name="kinect_pole_joint">
+    <origin xyz="0.275 0.0 0.1" rpy="0 0 0"/>
+    <child link="kinect_pole"/>
+    <parent link="chassis"/>
+  </joint>
+  <link name='kinect_pole'>
     <pose>0 0 0 0 0 0</pose>
     <inertial>
@@ -127,5 +127,5 @@
       </geometry>
     </collision>
-    <visual name='laser_pole_visual'>
+    <visual name='kinect_pole_visual'>
       <origin xyz="0 0.0 0.1" rpy=" 0 0 0"/>
         <geometry>
@@ -233,18 +233,5 @@
 -->
 <!-- Kinect Sensor -->
-<!-- link name must match the name of the reference in the .gazebo file -->
-    <link name="kinect_link">
-        <visual>
-            <origin xyz="0 0 0" rpy="0 0 1.5708"/>
-            <geometry>
-                <mesh filename="package://rtab_dumpster/meshes/kinect.dae" scale="1.0 1.0 1.0"/>
-            </geometry>
-        </visual>
-    </link>
-    <joint name="kinect_joint" type="fixed">
-        <origin xyz="0.0 0 0.285" rpy="0 0 0"/>
-        <parent link="laser_pole"/>
-        <child link="kinect_link"/>
-</joint>
+<xacro:include filename="$(find rtab_dumpster)/urdf/kinect.xacro"/>
 <!-- Laser -->
 <!--

Commit message: Add new laser pole and hokuyo laser sensor to robot model

File: urdf/rtab_dumpster.xacro (robot description, xacro)
@@ -59,5 +59,5 @@
 <!-- Dump box -->
     <joint name="dump_box_joint" type="fixed">
-    <origin xyz="0 0 0.1" rpy="1.57079 0 1.57079" />
+    <origin xyz="-0.025 0.0 0.1" rpy="1.57079 0 1.57079" /> <!-- X:front,back, Y:left,right, Z:up,down-->
     <parent link="chassis"/>
     <child link="dump_box" />
@@ -134,4 +134,34 @@
     </visual>
   </link>
+<!-- laser pole -->
+<joint type="fixed" name="laser_pole_joint">
+    <origin xyz="0.225 0.0 0.1" rpy="0 0 0"/>
+    <child link="laser_pole"/>
+    <parent link="chassis"/>
+  </joint>
+  <link name='laser_pole'>
+    <pose>0 0 0 0 0 0</pose>
+    <inertial>
+      <mass value="0.2"/>
+      <origin xyz="0.0 0 0" rpy=" 0 0 0"/>
+      <inertia
+          ixx="0.1" ixy="0" ixz="0"
+          iyy="0.1" iyz="0"
+          izz="0.1"
+      />
+    </inertial>
+    <collision name='collision'>
+      <origin xyz="0 0.0 0.1" rpy=" 0 0 0"/>
+      <geometry>
+        <box size="0.05 0.05 0.5"/>
+      </geometry>
+    </collision>
+    <visual name='laser_pole_visual'>
+      <origin xyz="0 0.0 0.1" rpy=" 0 0 0"/>
+        <geometry>
+        <box size="0.05 0.05 0.5"/>
+        </geometry>
+    </visual>
+  </link>
 <!-- Wheels -->
 <joint type="continuous" name="left_wheel_hinge">
@@ -235,5 +265,4 @@
 <xacro:include filename="$(find rtab_dumpster)/urdf/kinect.xacro"/>
 <!-- Laser -->
-<!--
 <link name="hokuyo">
     <pose>0 0 0.1 0 0 0</pose>
@@ -261,8 +290,7 @@
   </link>
 <joint type="fixed" name="hokuyo_joint">
-    <origin xyz="0.0 0 0.285" rpy="0 0 0"/>
+    <origin xyz="0.0 0 0.375" rpy="0 0 0"/>
     <child link="hokuyo"/>
     <parent link="laser_pole"/>
   </joint>
--->
 </robot>
