Commit message: Edit, make sure point cloud is correctly oriented to world in Rviz Edit, change camera_rgb_frame to camera_rgbd_frame Edit, make sure Kinect's mesh is correctly oriented Edit, align Kinect's base to the surface to which it is fixed

File: urdf/kinect.xacro (robot description, xacro)
@@ -1,13 +1,15 @@
 <?xml version="1.0"?>
 <robot name="sensor_kinect" xmlns:xacro="http://www.ros.org/wiki/xacro">
-  <xacro:property name="kinect_cam_py" value="-0.0125"/>
   <xacro:property name="M_PI" value="3.1415926535897931" />
-  	<xacro:property name="cam_px" value="0" />
-	<xacro:property name="cam_pz" value="0" />
-	<xacro:property name="cam_or" value="0" />
-	<xacro:property name="cam_op" value="0" />
-	<xacro:property name="cam_oy" value="0" />
+  <xacro:property name="cam_px" value="0" />
+  <xacro:property name="kinect_cam_py" value="0"/> <!-- distance of kinect base to surface to which it is fixed -->
+  <xacro:property name="cam_pz" value="0" />
+  <!-- change to make sure point cloud displayed in rviz is correctly alligned to world -->
+  <xacro:property name="cam_or" value="1.57079" />
+  <xacro:property name="cam_op" value="3.14159" />
+  <xacro:property name="cam_oy" value="1.57079" />
         <joint name="kinect_joint" type="fixed">
-        <origin xyz="0.04 0 0.3" rpy="0 0 0"/>
+        <!-- align kinect's base to the surface to which it is fixed -->
+        <origin xyz="0.012 0 0.285" rpy="0 0 0"/>
         <parent link="kinect_pole"/>
         <child link="kinect_baselink"/>
@@ -18,21 +20,23 @@
       <origin xyz="${cam_px} ${kinect_cam_py} ${cam_pz}" rpy="${cam_or} ${cam_op} ${cam_oy}"/>
       <parent link="kinect_baselink"/>
-      <child link="camera_rgb_frame" />
+      <child link="camera_rgbd_frame" />
     </joint>
-    <link name="camera_rgb_frame"/>
+    <link name="camera_rgbd_frame"/>
     <joint name="camera_rgb_optical_joint" type="fixed">
       <origin xyz="0 0 0" rpy="${-M_PI/2} 0 ${-M_PI/2}" />
-      <parent link="camera_rgb_frame" />
+      <parent link="camera_rgbd_frame" />
       <child link="camera_rgb_optical_frame" />
     </joint>
-    <link name="camera_rgb_optical_frame"/>\
-    <joint name="camera_joint" type="fixed">
-      <origin xyz="-0.031 ${-kinect_cam_py} -0.016" rpy="0 0 0"/>
-      <parent link="camera_rgb_frame"/>
-      <child link="camera_link"/>
+    <link name="camera_rgb_optical_frame"/>
+    <joint name="camera_meash_joint" type="fixed">
+      <origin xyz="0 ${-kinect_cam_py} 0" rpy="0 0 0"/>
+     <!-- <origin xyz="-0.031 ${-kinect_cam_py} -0.016" rpy="0 0 0"/> -->
+      <parent link="camera_rgbd_frame"/>
+      <child link="camera_mesh_link"/>
     </joint>
-      <link name="camera_link">
+      <link name="camera_mesh_link">
       <visual>
-       <origin xyz="0 0 0" rpy="0 0 ${M_PI/2}"/>
+      <!-- change to make sure mesh image is correctly rotated once depth could is rightly alligned -->
+       <origin xyz="0 0 0" rpy="-1.57079 0 3.14159"/>
         <geometry>
          <mesh filename="package://rtab_dumpster/meshes/kinect.dae" scale="1.0 1.0 1.0"/>
@@ -40,5 +44,5 @@
       </visual>
   	  <collision>
-        <origin xyz="0.0 0.0 0.0" rpy="0 0 0"/>
+        <origin xyz="0 0 0" rpy="-1.57079 0 3.14159"/>
   	    <geometry>
   	      <box size="0.07271 0.27794 0.073"/>
@@ -57,5 +61,5 @@
 	<joint name="camera_depth_joint" type="fixed">
 	  <origin xyz="0 ${2 * -kinect_cam_py} 0" rpy="0 0 0" />
-	  <parent link="camera_rgb_frame" />
+	  <parent link="camera_rgbd_frame" />
 	  <child link="camera_depth_frame" />
 	</joint>

Commit message: Refactor: iterate robot model design, exchange laser & kinect positions

File: urdf/kinect.xacro (robot description, xacro)
@@ -11,5 +11,5 @@
         <joint name="kinect_joint" type="fixed">
         <!-- align kinect's base to the surface to which it is fixed -->
-        <origin xyz="0.012 0 0.285" rpy="0 0 0"/>
+        <origin xyz="0 0 0.235" rpy="0 0 0"/> <!-- set height -->
         <parent link="kinect_pole"/>
         <child link="kinect_baselink"/>

File: urdf/rtab_dumpster.xacro (robot description, xacro)
@@ -2,5 +2,5 @@
 <robot name="rtab_dumpster" xmlns:xacro="http://www.ros.org/wiki/xacro">
 <xacro:include filename="$(find rtab_dumpster)/urdf/rtab_dumpster.gazebo" />
-  <link name="robot_footprint"></link>
+<link name="robot_footprint"></link>
 <!-- Chassis & caster wheels -->
   <joint name="robot_footprint_joint" type="fixed">
@@ -106,5 +106,6 @@
 <!-- kinect pole -->
 <joint type="fixed" name="kinect_pole_joint">
-    <origin xyz="0.275 0.0 0.1" rpy="0 0 0"/>
+<!--    <origin xyz="0.275 0.0 0.1" rpy="0 0 0"/> -->
+    <origin xyz="0.225 0.0 0.05" rpy="0 0 0"/>
     <child link="kinect_pole"/>
     <parent link="chassis"/>
@@ -124,5 +125,5 @@
       <origin xyz="0 0.0 0.1" rpy=" 0 0 0"/>
       <geometry>
-        <box size="0.05 0.05 0.3"/>
+        <box size="0.05 0.05 0.2"/>
       </geometry>
     </collision>
@@ -130,5 +131,5 @@
       <origin xyz="0 0.0 0.1" rpy=" 0 0 0"/>
         <geometry>
-        <box size="0.05 0.05 0.3"/>
+        <box size="0.05 0.05 0.2"/>
         </geometry>
     </visual>
@@ -136,5 +137,6 @@
 <!-- laser pole -->
 <joint type="fixed" name="laser_pole_joint">
-    <origin xyz="0.225 0.0 0.1" rpy="0 0 0"/>
+   <!-- <origin xyz="0.225 0.0 0.1" rpy="0 0 0"/> -->
+    <origin xyz="0.275 0.0 0.05" rpy="0 0 0"/>
     <child link="laser_pole"/>
     <parent link="chassis"/>
@@ -152,13 +154,13 @@
     </inertial>
     <collision name='collision'>
-      <origin xyz="0 0.0 0.1" rpy=" 0 0 0"/>
-      <geometry>
-        <box size="0.05 0.05 0.5"/>
+      <origin xyz="0 0.0 0.05" rpy=" 0 0 0"/>
+      <geometry>
+        <box size="0.05 0.05 0.1"/>
       </geometry>
     </collision>
     <visual name='laser_pole_visual'>
-      <origin xyz="0 0.0 0.1" rpy=" 0 0 0"/>
+      <origin xyz="0 0 0.05" rpy=" 0 0 0"/>
         <geometry>
-        <box size="0.05 0.05 0.5"/>
+        <box size="0.05 0.05 0.1"/>
         </geometry>
     </visual>
@@ -266,5 +268,5 @@
 <!-- Laser -->
 <link name="hokuyo">
-    <pose>0 0 0.1 0 0 0</pose>
+    <pose>0 0 0 0 0 0</pose>
     <inertial>
       <mass value="0.1"/>
@@ -290,5 +292,5 @@
   </link>
 <joint type="fixed" name="hokuyo_joint">
-    <origin xyz="0.0 0 0.375" rpy="0 0 0"/>
+    <origin xyz="0.0 0 0.135" rpy="0 0 0"/> <!-- set height relative to laser_pole -->
     <child link="hokuyo"/>
     <parent link="laser_pole"/>
